File: inputstage.kicad_sch (KiCad schematic)
At the start: 8 parts, among them J1 HV_IN_P, J2 HV_IN_N

Commit message: Updated schematic and fixed silkscreen overlap
Parts:
- L1: value 1 -> 2
Changed lines of the file:
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@@
       (effects (font (size 1.27 1.27)))
     )
-    (property "Value" "1" (at 158.75 50.8 90)
+    (property "Value" "2" (at 158.75 50.8 90)
       (effects (font (size 1.27 1.27)))
     )

Commit message: Added footprint
Parts:
- F1: footprint (none) -> 100nf:100NF CAPC1005X55N
Changed lines of the file:
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@@
       (effects (font (size 1.27 1.27)))
     )
-    (property "Footprint" "" (at 123.19 55.118 90)
+    (property "Footprint" "100nf:100NF CAPC1005X55N" (at 123.19 55.118 90)
       (effects (font (size 1.27 1.27)) hide)
     )

Commit message: Updated schematic and added RS485 protection circuit
Parts:
- removed J1: HV_IN_P, symbol Connector:Screw_Terminal_01x01
- removed J2: HV_IN_N, symbol Connector:Screw_Terminal_01x01
- L1: value 2 -> 1
Connections:
- net HV_IN_P: now reaches Rf1.1
- net VIN_MINUS renamed HV_IN_N
Changed lines of the file:
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@@
     (stroke (width 0) (type default))
+  )
+  (hierarchical_label "HV_IN_N" (shape input) (at 110.49 90.17 180) (fields_autoplaced)
+    (effects (font (size 1.27 1.27)) (justify right))
+  )
+  (hierarchical_label "HV_IN_P" (shape input) (at 105.41 53.34 180) (fields_autoplaced)
+    (effects (font (size 1.27 1.27)) (justify right))
   )
   (hierarchical_label "HV_BULK_+" (shape output) (at 185.42 53.34 0) (fields_autoplaced)
@@
     )
   )
-  (symbol (lib_id "Connector:Screw_Terminal_01x01") (at 100.33 53.34 0) (mirror y) (unit 1)
-    (in_bom yes) (on_board yes) (dnp no)
-    (property "Reference" "J1" (at 97.79 52.07 0)
-      (effects (font (size 1.27 1.27)) (justify left))
-    )
-    (property "Value" "HV_IN_P" (at 97.79 54.61 0)
-      (effects (font (size 1.27 1.27)) (justify left))
-    )
-    (property "Footprint" "" (at 100.33 53.34 0)
-      (effects (font (size 1.27 1.27)) hide)
-    )
-    (property "Datasheet" "~" (at 100.33 53.34 0)
-      (effects (font (size 1.27 1.27)) hide)
-    )
-    (property "Sim.Enable" "0" (at 100.33 53.34 0)
-      (effects (font (size 1.27 1.27)) hide)
-    )
-    (pin "1")
-    (instances
-      (project "UC28881  WORK"
-        (path "/02261b3b-0ab5-411c-b90d-2981c1ef32c1/fb27a4d2-e43a-4d93-b9d6-c1683e793fef"
-          (reference "J1") (unit 1)
-        )
-      )
-    )
-  )
-  (symbol (lib_id "Connector:Screw_Terminal_01x01") (at 105.41 90.17 180) (unit 1)
-    (in_bom yes) (on_board yes) (dnp no)
-    (property "Reference" "J2" (at 106.1339 93.98 90)
-      (effects (font (size 1.27 1.27)) (justify left))
-    )
-    (property "Value" "HV_IN_N" (at 103.5939 93.98 90)
-      (effects (font (size 1.27 1.27)) (justify left))
-    )
-    (property "Footprint" "" (at 105.41 90.17 0)
-      (effects (font (size 1.27 1.27)) hide)
-    )
-    (property "Datasheet" "~" (at 105.41 90.17 0)
-      (effects (font (size 1.27 1.27)) hide)
-    )
-    (pin "1")
-    (instances
-      (project "UC28881  WORK"
-        (path "/02261b3b-0ab5-411c-b90d-2981c1ef32c1/fb27a4d2-e43a-4d93-b9d6-c1683e793fef"
-          (reference "J2") (unit 1)
-        )
-      )
-    )
-  )
   (symbol (lib_id "Device:R") (at 109.22 53.34 90) (unit 1)
     (in_bom yes) (on_board yes) (dnp no) (fields_autoplaced)
@@
       (effects (font (size 1.27 1.27)))
     )
-    (property "Value" "2" (at 158.75 50.8 90)
+    (property "Value" "1" (at 158.75 50.8 90)
       (effects (font (size 1.27 1.27)))
     )
