File: _autosave-UC28881  WORK.kicad_sch (KiCad schematic)
At the start: 18 parts, among them J1 Screw_Terminal_01x02, J2 Screw_Terminal_01x02, U1 UCC28881

Commit message: Initial commit
Parts:
- D2: footprint Diode_SMD:D_1206_3216Metric -> D2:D2
Changed lines of the file:
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@@
       (effects (font (size 1.27 1.27)) (justify left))
     )
-    (property "Footprint" "Diode_SMD:D_1206_3216Metric" (at 231.14 57.15 0)
+    (property "Footprint" "D2:D2" (at 231.14 57.15 0)
       (effects (font (size 1.27 1.27)) hide)
     )
