File: _autosave-UC28881  WORK.kicad_pcb (KiCad board)
At the start: 2 copper layers, 102 x 50 mm, 22 parts, among them J1 Screw_Terminal_01x02, J2 Screw_Terminal_01x02, U1 UCC28881

Commit message: Initial commit
Parts:
- removed the REF** at (76.2, 38.1)
- removed the REF** at (169.0, 78.7)
- removed the REF** at (76.2, 78.7)
- removed the REF** at (168.9, 38.1)
- added REF**: MountingHole_3.2mm_M3_DIN965, MountingHole:MountingHole_3.2mm_M3_DIN965, F.Cu at (73.7, 38.1)
- D2: footprint Diode_SMD:D_1206_3216Metric -> D2:D2
- moved Rf1 1.98 mm to (80.0, 40.6)
- moved D2 0.82 mm to (138.4, 63.5), turned to 0 degrees
Routing:
- net /10V_OUT_P: track 66.1 -> 55.8 mm

Commit message: updated
Parts:
- removed the REF** at (73.7, 38.1)
- added REF**: MountingHole_3.2mm_M3_DIN965_Pad, MountingHole:MountingHole_3.2mm_M3_DIN965_Pad, F.Cu at (74.9, 38.1)
- added REF**: MountingHole_3.2mm_M3_DIN965_Pad, MountingHole:MountingHole_3.2mm_M3_DIN965_Pad, F.Cu at (168.9, 80.0)
- added REF**: MountingHole_3.2mm_M3_DIN965_Pad, MountingHole:MountingHole_3.2mm_M3_DIN965_Pad, F.Cu at (74.9, 80.0)
- added REF**: MountingHole_3.2mm_M3_DIN965_Pad, MountingHole:MountingHole_3.2mm_M3_DIN965_Pad, F.Cu at (168.9, 38.1)
Changed lines of the file:
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@@
   (net 9 "unconnected-(U1-NC-Pad6)")
   (net 10 "/GND")
+  (footprint "MountingHole:MountingHole_3.2mm_M3_DIN965_Pad" (layer "F.Cu")
+    (at 74.93 38.1)
+    (descr "Mounting Hole 3.2mm, M3, DIN965")
+    (tags "mounting hole 3.2mm m3 din965")
+    (attr exclude_from_pos_files exclude_from_bom)
+    (fp_text reference "REF**" (at -7.62 -1.27) (layer "F.SilkS") hide
+        (effects (font (size 1 1) (thickness 0.15)))
+    )
+    (fp_text value "MountingHole_3.2mm_M3_DIN965_Pad" (at 0 3.8) (layer "F.Fab")
+        (effects (font (size 1 1) (thickness 0.15)))
+    )
+    (fp_text user "${REFERENCE}" (at 0 0) (layer "F.Fab")
+        (effects (font (size 1 1) (thickness 0.15)))
+    )
+    (fp_circle (center 0 0) (end 2.8 0)
+      (stroke (width 0.15) (type solid)) (fill none) (layer "Cmts.User"))
+    (fp_circle (center 0 0) (end 3.05 0)
+      (stroke (width 0.05) (type solid)) (fill none) (layer "F.CrtYd"))
+    (pad "1" thru_hole circle (at 0 0) (size 5.6 5.6) (drill 3.2) (layers "*.Cu" "*.Mask"))
+  )
   (footprint "C2:CAPC3225X88N" (layer "F.Cu")
     (at 122.1065 51.62 90)
@@
     )
   )
+  (footprint "MountingHole:MountingHole_3.2mm_M3_DIN965_Pad" (layer "F.Cu")
+    (at 168.91 80.01)
+    (descr "Mounting Hole 3.2mm, M3, DIN965")
+    (tags "mounting hole 3.2mm m3 din965")
+    (attr exclude_from_pos_files exclude_from_bom)
+    (fp_text reference "REF**" (at -7.62 -1.27) (layer "F.SilkS") hide
+        (effects (font (size 1 1) (thickness 0.15)))
+    )
+    (fp_text value "MountingHole_3.2mm_M3_DIN965_Pad" (at 0 3.8) (layer "F.Fab")
+        (effects (font (size 1 1) (thickness 0.15)))
+    )
+    (fp_text user "${REFERENCE}" (at 0 0) (layer "F.Fab")
+        (effects (font (size 1 1) (thickness 0.15)))
+    )
+    (fp_circle (center 0 0) (end 2.8 0)
+      (stroke (width 0.15) (type solid)) (fill none) (layer "Cmts.User"))
+    (fp_circle (center 0 0) (end 3.05 0)
+      (stroke (width 0.05) (type solid)) (fill none) (layer "F.CrtYd"))
+    (pad "1" thru_hole circle (at 0 0) (size 5.6 5.6) (drill 3.2) (layers "*.Cu" "*.Mask"))
+  )
   (footprint "C4:CAP_ECHU1H104GX9" (layer "F.Cu")
     (at 130.4565 62.63 180)
@@
       (rotate (xyz 90 180 0))
     )
+  )
+  (footprint "MountingHole:MountingHole_3.2mm_M3_DIN965_Pad" (layer "F.Cu")
+    (at 74.93 80.01)
+    (descr "Mounting Hole 3.2mm, M3, DIN965")
+    (tags "mounting hole 3.2mm m3 din965")
+    (attr exclude_from_pos_files exclude_from_bom)
+    (fp_text reference "REF**" (at -7.62 -1.27) (layer "F.SilkS") hide
+        (effects (font (size 1 1) (thickness 0.15)))
+    )
+    (fp_text value "MountingHole_3.2mm_M3_DIN965_Pad" (at 0 3.8) (layer "F.Fab")
+        (effects (font (size 1 1) (thickness 0.15)))
+    )
+    (fp_text user "${REFERENCE}" (at 0 0) (layer "F.Fab")
+        (effects (font (size 1 1) (thickness 0.15)))
+    )
+    (fp_circle (center 0 0) (end 2.8 0)
+      (stroke (width 0.15) (type solid)) (fill none) (layer "Cmts.User"))
+    (fp_circle (center 0 0) (end 3.05 0)
+      (stroke (width 0.05) (type solid)) (fill none) (layer "F.CrtYd"))
+    (pad "1" thru_hole circle (at 0 0) (size 5.6 5.6) (drill 3.2) (layers "*.Cu" "*.Mask"))
+  )
+  (footprint "MountingHole:MountingHole_3.2mm_M3_DIN965_Pad" (layer "F.Cu")
+    (at 168.91 38.1)
+    (descr "Mounting Hole 3.2mm, M3, DIN965")
+    (tags "mounting hole 3.2mm m3 din965")
+    (attr exclude_from_pos_files exclude_from_bom)
+    (fp_text reference "REF**" (at -7.62 -1.27) (layer "F.SilkS") hide
+        (effects (font (size 1 1) (thickness 0.15)))
+    )
+    (fp_text value "MountingHole_3.2mm_M3_DIN965_Pad" (at 0 3.8) (layer "F.Fab")
+        (effects (font (size 1 1) (thickness 0.15)))
+    )
+    (fp_text user "${REFERENCE}" (at 0 0) (layer "F.Fab")
+        (effects (font (size 1 1) (thickness 0.15)))
+    )
+    (fp_circle (center 0 0) (end 2.8 0)
+      (stroke (width 0.15) (type solid)) (fill none) (layer "Cmts.User"))
+    (fp_circle (center 0 0) (end 3.05 0)
+      (stroke (width 0.05) (type solid)) (fill none) (layer "F.CrtYd"))
+    (pad "1" thru_hole circle (at 0 0) (size 5.6 5.6) (drill 3.2) (layers "*.Cu" "*.Mask"))
   )
   (footprint "Diode_THT:D_DO-41_SOD81_P10.16mm_Horizontal" (layer "F.Cu")
@@
       (net 7 "/10V_OUT_P") (pinfunction "A") (pintype "passive"))
   )
-  (footprint "MountingHole:MountingHole_3.2mm_M3_DIN965" (layer "F.Cu")
-    (at 73.66 38.1)
-    (descr "Mounting Hole 3.2mm, no annular, M3, DIN965")
-    (tags "mounting hole 3.2mm no annular m3 din965")
-    (attr through_hole exclude_from_pos_files exclude_from_bom)
-    (fp_text reference "REF**" (at 0 -3.8) (layer "F.SilkS")
-        (effects (font (size 1 1) (thickness 0.15)))
-    )
-    (fp_text value "MountingHole_3.2mm_M3_DIN965" (at 0 3.8) (layer "F.Fab")
-        (effects (font (size 1 1) (thickness 0.15)))
-    )
-    (fp_circle (center 0 0) (end 2.8 0)
-      (stroke (width 0.15) (type solid)) (fill none) (layer "Cmts.User"))
-    (fp_circle (center 0 0) (end 3.05 0)
-      (stroke (width 0.05) (type solid)) (fill none) (layer "F.CrtYd"))
-    (pad "" np_thru_hole circle (at 0 0) (size 3.2 3.2) (drill 3.2) (layers "*.Cu" "*.Mask"))
-  )
   (footprint "88.7k resistor:ERJS1T_U1T__2512_" (layer "F.Cu")
