File: UC28881  WORK.kicad_pcb (KiCad board)
At the start: 2 copper layers, 102 x 50 mm, 22 parts, among them J1 Screw_Terminal_01x02, J2 Screw_Terminal_01x02, U1 UCC28881

Commit message: Updated PCB
Parts:
- removed CL1: 330u, CL1:CAP_UAQ_18X20_NCH
- removed D3: 1N5819, Diode_THT:D_DO-41_SOD81_P10.16mm_Horizontal
- removed J2: Screw_Terminal_01x02, TerminalBlock_Phoenix:TerminalBlock_Phoenix_MKDS-1,5-2_1x02_P5.00mm_Horizontal
- removed REF** (x4): MountingHole_3.2mm_M3_DIN965_Pad, MountingHole:MountingHole_3.2mm_M3_DIN965_Pad
- removed TVS1: D_Zener, TVS1:1.5KESeries_LTF
- added H1: MountingHole, MountingHole:MountingHole_3.2mm_M3_DIN965, F.Cu at (76.2, 69.8)
- added H2: MountingHole, MountingHole:MountingHole_3.2mm_M3_DIN965, F.Cu at (111.9, 69.8)
- added H3: MountingHole, MountingHole:MountingHole_3.2mm_M3_DIN965, F.Cu at (111.8, 38.1)
- added H4: MountingHole, MountingHole:MountingHole_3.2mm_M3_DIN965, F.Cu at (76.2, 38.1)
- C1: footprint Capacitor_THT:CP_Radial_D12.5mm_P7.50mm -> Capacitor_THT:CP_Radial_D10.0mm_P5.00mm
- D1: footprint Diode_THT:D_DO-35_SOD27_P7.62mm_Horizontal -> D1:SMA_STM-M
- D2: value SS1P3L -> M7; footprint Diode_SMD:D_1206_3216Metric -> D2:D2
- J1: value Screw_Terminal_01x02 -> Screw_Terminal_01x03; footprint TerminalBlock_Phoenix:TerminalBlock_Phoenix_MKDS-1,5-2_1x02_P5.00mm_Horizontal -> TerminalBlock_Phoenix:TerminalBlock_Phoenix_MKDS-1,5-3-5.08_1x03_P5.08mm_Horizontal
- RFB1: footprint 10k resistor:10k RES_3540_TEC-M -> 10k resistor:10k RESC1005X35N
- RFB2: value 87.7K -> 110k; footprint 88.7k resistor:ERJS1T_U1T__2512_ -> 110k resistor:110k RESC1005X35N
- Rf1: footprint Resistor_THT:R_Axial_DIN0922_L20.0mm_D9.0mm_P30.48mm_Horizontal -> RF:ERJUP6
- moved L2 51.9 mm to (101.5, 64.8), turned to 180 degrees
- moved D1 35.8 mm to (99.1, 53.0)
- moved D2 34.2 mm to (104.8, 55.9), turned to 0 degrees
- moved RFB2 32.2 mm to (105.0, 46.9), turned to -90 degrees
- moved C3 29.1 mm to (98.3, 47.9)
- moved U1 27.8 mm to (103.8, 42.8)
- moved C2 26.8 mm to (96.8, 42.9)
- moved C4 24.4 mm to (108.2, 52.7)
- moved RFB1 24.3 mm to (102.9, 47.0), turned to -90 degrees
- moved C1 22.3 mm to (92.5, 51.9)
- moved L1 17.0 mm to (84.9, 39.9)
- moved CBULK1 6.58 mm to (89.1, 67.0), turned to 90 degrees
- moved Rf1 5.66 mm to (77.6, 45.7)
- moved J1 3.81 mm to (77.5, 50.8)
Connections:
- J1 pad 1: /HV_IN_P -> /10V_OUT_P
Routing:
- net Net-(U1-DRAIN): track 86.3 -> 43.5 mm
- net /Feedback pin: track 17.8 -> 44.2 mm
- net /GND: track 33.6 -> 10.4 mm
- net /10V_OUT_P: track 66.1 -> 56.9 mm
- net Net-(CBULK1-Pad1): track 48.5 -> 55.6 mm
- net Net-(D2-K): track 14.6 -> 17.9 mm
- net /HV_IN_P: track 13.8 -> 16.2 mm
- net Net-(D1-K): track 62.1 -> 60.3 mm
- net Net-(U1-VDD): track 6.12 -> 4.51 mm
Other:
- board size 102 x 50 mm -> 44.7 x 41.3 mm

Commit message: update
Parts:
- L1: footprint L1 1MH:IND_EPCOS_B82472G6_EPC -> L1 1MH:L_Wurth_WE-PD2HV-7850
- RFB1: footprint 10k resistor:10k RESC1005X35N -> 10k resistor:RESC3116X65N
- RFB2: footprint 110k resistor:110k RESC1005X35N -> 110k resistor:RESC3216X75N
- Rf1: value 10 -> 15; footprint RF:ERJUP6 -> RF:RF1 RC1206N_PAN-M
- moved RFB2 2.28 mm to (107.1, 47.9)
- moved RFB1 1.08 mm to (103.5, 47.9)
Routing:
- net Net-(D1-K): track 60.3 -> 75.1 mm
- net Net-(D2-K): track 17.9 -> 14.0 mm
- net /Feedback pin: track 44.2 -> 46.9 mm
- net Net-(CBULK1-Pad1): track 55.6 -> 53.3 mm
- net /HV_IN_P: track 16.2 -> 17.6 mm
- net Net-(U1-DRAIN): track 43.5 -> 42.4 mm
- net /10V_OUT_P: track 56.9 -> 57.8 mm

Commit message: update
Parts:
- added COUT1: 47UF, Capacitor_SMD:C_1206_3216Metric_Pad1.33x1.80mm_HandSolder, F.Cu at (111.1, 56.3)
- D1: value 1N4148 -> STTH1R06A
Routing:
- net /10V_OUT_P: track 57.8 -> 66.3 mm
- net /GND: track 10.4 -> 12.7 mm, vias 0 -> 1
Changed lines of the file:
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@@
         (effects (font (size 1 1) (thickness 0.15)))
     )
-    (fp_text value "1N4148" (at -0.13 -0.16 180 unlocked) (layer "F.Fab")
+    (fp_text value "STTH1R06A" (at -0.13 -0.16 180 unlocked) (layer "F.Fab")
         (effects (font (size 1 1) (thickness 0.15)))
     )
@@
     (property "ki_keywords" "inductor choke coil reactor magnetic")
     (attr smd)
-    (fp_text reference "L1" (at 0 -5 unlocked) (layer "F.SilkS")
+    (fp_text reference "L1" (at -1.03 -4.77 unlocked) (layer "F.SilkS")
         (effects (font (size 1 1) (thickness 0.15)))
     )
@@
       (net 1 "Net-(U1-DRAIN)") (pinfunction "2") (pintype "passive"))
     (model "${KIPRJMOD}/3D models/L1   L_Wurth_WE-PD2HV-7850.step"
+      (offset (xyz 0 0 0))
+      (scale (xyz 1 1 1))
+      (rotate (xyz 0 0 0))
+    )
+  )
+  (footprint "Capacitor_SMD:C_1206_3216Metric_Pad1.33x1.80mm_HandSolder" (layer "F.Cu")
+    (at 111.1425 56.34 180)
+    (descr "Capacitor SMD 1206 (3216 Metric), square (rectangular) end terminal, IPC_7351 nominal with elongated pad for handsoldering. (Body size source: IPC-SM-782 page 76, https://www.pcb-3d.com/wordpress/wp-content/uploads/ipc-sm-782a_amendment_1_and_2.pdf), generated with kicad-footprint-generator")
+    (tags "capacitor handsolder")
+    (property "PART NUMBER" "C3216X5R1C476M160AB")
+    (property "Sheetfile" "UC28881  WORK.kicad_sch")
+    (property "Sheetname" "")
+    (property "ki_description" "Unpolarized capacitor")
+    (property "ki_keywords" "cap capacitor")
+    (attr smd)
+    (fp_text reference "COUT1" (at -0.4575 -1.88) (layer "F.SilkS")
+        (effects (font (size 1 1) (thickness 0.15)))
+    )
+    (fp_text value "47UF" (at -2.5375 2.23) (layer "F.Fab")
+        (effects (font (size 1 1) (thickness 0.15)))
+    )
+    (fp_text user "${REFERENCE}" (at 0 0) (layer "F.Fab")
+        (effects (font (size 0.8 0.8) (thickness 0.12)))
+    )
+    (fp_line (start -0.711252 -0.91) (end 0.711252 -0.91)
+      (stroke (width 0.12) (type solid)) (layer "F.SilkS"))
+    (fp_line (start -0.711252 0.91) (end 0.711252 0.91)
+      (stroke (width 0.12) (type solid)) (layer "F.SilkS"))
+    (fp_line (start -2.48 -1.15) (end 2.48 -1.15)
+      (stroke (width 0.05) (type solid)) (layer "F.CrtYd"))
+    (fp_line (start -2.48 1.15) (end -2.48 -1.15)
+      (stroke (width 0.05) (type solid)) (layer "F.CrtYd"))
+    (fp_line (start 2.48 -1.15) (end 2.48 1.15)
+      (stroke (width 0.05) (type solid)) (layer "F.CrtYd"))
+    (fp_line (start 2.48 1.15) (end -2.48 1.15)
+      (stroke (width 0.05) (type solid)) (layer "F.CrtYd"))
+    (fp_line (start -1.6 -0.8) (end 1.6 -0.8)
+      (stroke (width 0.1) (type solid)) (layer "F.Fab"))
+    (fp_line (start -1.6 0.8) (end -1.6 -0.8)
+      (stroke (width 0.1) (type solid)) (layer "F.Fab"))
+    (fp_line (start 1.6 -0.8) (end 1.6 0.8)
+      (stroke (width 0.1) (type solid)) (layer "F.Fab"))
+    (fp_line (start 1.6 0.8) (end -1.6 0.8)
+      (stroke (width 0.1) (type solid)) (layer "F.Fab"))
+    (pad "1" smd roundrect (at -1.5625 0 180) (size 1.325 1.8) (layers "F.Cu" "F.Paste" "F.Mask") (roundrect_rratio 0.188679)
+      (net 6 "/10V_OUT_P") (pintype "passive"))
+    (pad "2" smd roundrect (at 1.5625 0 180) (size 1.325 1.8) (layers "F.Cu" "F.Paste" "F.Mask") (roundrect_rratio 0.188679)
+      (net 9 "/GND") (pintype "passive"))
+    (model "${KICAD6_3DMODEL_DIR}/Capacitor_SMD.3dshapes/C_1206_3216Metric.wrl"
       (offset (xyz 0 0 0))
       (scale (xyz 1 1 1))
@@
   (segment (start 77.47 50.795) (end 82.545 50.795) (width 0.5) (layer "F.Cu") (net 6))
   (segment (start 105.6155 71.2176) (end 109.89 66.9431) (width 0.5) (layer "F.Cu") (net 6))
+  (segment (start 114.28 59.17) (end 113.47 59.98) (width 0.5) (layer "F.Cu") (net 6))
   (segment (start 109.89 66.9431) (end 109.89 59.6) (width 0.5) (layer "F.Cu") (net 6))
   (segment (start 96.52 64.77) (end 96.52 69.339954) (width 0.5) (layer "F.Cu") (net 6))
+  (segment (start 114.28 57.66) (end 114.28 59.17) (width 0.5) (layer "F.Cu") (net 6))
   (segment (start 96.52 69.339954) (end 98.397646 71.2176) (width 0.5) (layer "F.Cu") (net 6))
+  (segment (start 113.47 59.98) (end 110.27 59.98) (width 0.5) (layer "F.Cu") (net 6))
+  (segment (start 112.705 56.34) (end 112.96 56.34) (width 0.5) (layer "F.Cu") (net 6))
   (segment (start 82.545 50.795) (end 96.52 64.77) (width 0.5) (layer "F.Cu") (net 6))
+  (segment (start 110.27 59.98) (end 109.89 59.6) (width 0.5) (layer "F.Cu") (net 6))
+  (segment (start 112.96 56.34) (end 114.28 57.66) (width 0.5) (layer "F.Cu") (net 6))
   (segment (start 109.89 59.6) (end 106.295 56.005) (width 0.5) (layer "F.Cu") (net 6))
   (segment (start 74.06 57.545) (end 74.06 48.05) (width 0.5) (layer "F.Cu") (net 7))
@@
   (segment (start 77.47 60.955) (end 74.06 57.545) (width 0.5) (layer "F.Cu") (net 7))
   (segment (start 97.1488 52.95) (end 96.7988 53.3) (width 0.5) (layer "F.Cu") (net 9))
+  (segment (start 108.51 56.34) (end 108.21 56.04) (width 0.5) (layer "F.Cu") (net 9))
+  (segment (start 109.58 56.34) (end 108.51 56.34) (width 0.5) (layer "F.Cu") (net 9))
   (segment (start 96.7988 53.3) (end 88.99 53.3) (width 0.5) (layer "F.Cu") (net 9))
   (segment (start 88.99 53.3) (end 87.54 51.85) (width 0.5) (layer "F.Cu") (net 9))
+  (via (at 108.21 56.04) (size 0.6) (drill 0.3) (layers "F.Cu" "B.Cu") (net 9))
+  (segment (start 107.68 55.51) (end 107.59 55.51) (width 0.5) (layer "B.Cu") (net 9))
+  (segment (start 108.21 56.04) (end 107.68 55.51) (width 0.5) (layer "B.Cu") (net 9))
   (segment (start 78.74 45.72) (end 78.74 43.28) (width 0.5) (layer "F.Cu") (net 10))
   (segment (start 78.12 42.66) (end 78.74 43.28) (width 0.5) (layer "F.Cu") (net 10))

Commit message: edited pcb layout
Parts:
- C2: value 0.1u -> (none)
- COUT1: value 47UF -> (none)
- D2: value M7 -> (none)
- RFB2: value 110k -> (none)
- U1: value UCC28881 -> (none)
- moved CBULK1 27.6 mm to (93.9, 39.8), turned to 0 degrees
- moved C2 19.2 mm to (100.9, 61.6), turned to 180 degrees
- moved C1 16.4 mm to (85.0, 37.2), turned to -90 degrees
- moved Rf1 14.9 mm to (86.6, 57.6)
- moved D1 13.9 mm to (112.8, 50.6), turned to -90 degrees
- moved L2 11.4 mm to (90.3, 66.9)
- moved L1 11.1 mm to (88.0, 50.5), turned to 180 degrees
- moved C3 10.6 mm to (108.6, 49.9), turned to 90 degrees
- moved RFB2 10.4 mm to (106.5, 58.3), turned to 180 degrees
- moved COUT1 10.2 mm to (101.0, 55.4), turned to 0 degrees
- moved C4 9.28 mm to (107.2, 61.9), turned to 0 degrees
- moved RFB1 8.01 mm to (106.4, 55.3), turned to 180 degrees
- moved U1 6.70 mm to (102.2, 49.3)
- moved D2 4.58 mm to (100.9, 58.4), turned to 180 degrees
- moved J1 1.27 mm to (77.5, 49.5)
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Routing:
- net Net-(CBULK1-Pad1): track 53.3 -> 20.3 mm
- net /Feedback pin: track 46.9 -> 19.8 mm, vias 0 -> 2
- net /GND: track 12.7 -> 37.5 mm, vias 1 -> 2
- net /10V_OUT_P: track 66.3 -> 43.8 mm
- net Net-(D1-K): track 75.1 -> 56.5 mm
- net Net-(U1-VDD): track 4.51 -> 19.1 mm, vias 0 -> 2
- net /HV_IN_P: track 17.6 -> 9.02 mm, vias 0 -> 1
- net Net-(D2-K): track 14.0 -> 6.33 mm
- net Net-(U1-DRAIN): track 42.4 -> 43.8 mm, vias 0 -> 2

Commit message: ADDED BOM
Parts:
- C2: value (none) -> 0.1u; footprint C2:CAPC3225X88N -> Capacitor_SMD:C_1206_3216Metric
- C3: footprint C3:CAP_ECHU1H104GX9 -> Capacitor_SMD:C_1206_3216Metric
- C4: footprint C4:CAP_ECHU1H104GX9 -> Capacitor_SMD:C_1206_3216Metric
- COUT1: value (none) -> 47UF
- D2: value (none) -> M7
- RFB2: value (none) -> 110k
- U1: value (none) -> UCC28881
- moved C4 0.77 mm to (106.4, 61.6)
Routing:
- net Net-(D1-K): track 56.5 -> 58.0 mm

Commit message: update
Connections:
- net /10V_OUT_P renamed /12V_OUT_P
Other:
- board text added: "12V"
- board text added: "GND"
- board text added: "HV_IN"
Changed lines of the file:
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@@
   (net 4 "/Feedback pin")
   (net 5 "Net-(D2-K)")
-  (net 6 "/10V_OUT_P")
+  (net 6 "/12V_OUT_P")
   (net 7 "/HV_IN_P")
   (net 8 "unconnected-(U1-NC-Pad6)")
@@
     (tags "capacitor")
     (property "MANUFACTURER" "KYOCERA AVX")
-    (property "MANUFACTURER PART NUMBER" "12065C104JAT2A")
-    (property "PACKAGE " "1206")
+    (property "MANUFACTURER PART NO" "12065C104JAT2A")
+    (property "PACKAGE" "1206")
     (property "SUPPLIER" "MOUSER")
     (property "SUPPLIER PART NO" "581-12065C104J")
@@
       (stroke (width 0.1) (type solid)) (fill none) (layer "F.Fab"))
     (pad "1" thru_hole rect (at 0 0 270) (size 2.6 2.6) (drill 1.3) (layers "*.Cu" "*.Mask")
-      (net 6 "/10V_OUT_P") (pinfunction "Pin_1") (pintype "passive"))
+      (net 6 "/12V_OUT_P") (pinfunction "Pin_1") (pintype "passive"))
     (pad "2" thru_hole circle (at 5.08 0 270) (size 2.6 2.6) (drill 1.3) (layers "*.Cu" "*.Mask")
       (net 9 "/GND") (pinfunction "Pin_2") (pintype "passive"))
@@
     (descr "TI SOIC‑8 (D), P1.27 mm, pads 1.55×0.60 mm, row spacing 5.40 mm — UCC28881 land pattern (per TI datasheet)")
     (tags "SOIC-8 D 1.27mm UCC28881 UC28881 TI")
-    (property "MANUFACTURER " "TEXAS INSTRUMENTS")
+    (property "MANUFACTURER" "TEXAS INSTRUMENTS")
     (property "MANUFACTURER PART NO" "UCC28810D")
-    (property "PACKAGE " "8-SOIC")
+    (property "PACKAGE" "8-SOIC")
     (property "SUPPLIER" "DIGIKEY")
     (property "SUPPLIER PART NO" "296-27162-5-ND")
@@
     (property "MANUFACTURER PART NO" "CR2010-FX-1002ELF")
     (property "PACKAGE" "2010")
-    (property "SUPLLIER" "DIGIKEY")
+    (property "SUPPLIER" "DIGIKEY")
     (property "SUPPLIER PART NO" "118-CR2010-FX-1002ELFCT-ND")
     (property "Sheetfile" "UC28881  WORK.kicad_sch")
@@
     (descr "Unhielded Power Inductor (High Voltage), body 7.8x7x4.9mm, https://www.we-online.com/en/components/products/WE-PD2-HV#/articles/WE-PD2-HV-7850")
     (tags "SMT")
-    (property "DNP" "YES")
-    (property "MANUFACTURER PART NUMBER" "76877530")
+    (property "MANUFACTURER" ".")
+    (property "MANUFACTURER PART NO" "76877530")
+    (property "SUPPLIER" ".")
+    (property "SUPPLIER PART NO" ".")
     (property "Sheetfile" "UC28881  WORK.kicad_sch")
     (property "Sheetname" "")
@@
       (stroke (width 0.1) (type solid)) (layer "F.Fab"))
     (pad "1" smd roundrect (at -1.5625 0) (size 1.325 1.8) (layers "F.Cu" "F.Paste" "F.Mask") (roundrect_rratio 0.188679)
-      (net 6 "/10V_OUT_P") (pintype "passive"))
+      (net 6 "/12V_OUT_P") (pintype "passive"))
     (pad "2" smd roundrect (at 1.5625 0) (size 1.325 1.8) (layers "F.Cu" "F.Paste" "F.Mask") (roundrect_rratio 0.188679)
       (net 9 "/GND") (pintype "passive"))
@@
   (footprint "D2:D2" (layer "F.Cu")
     (at 100.945 58.405 180)
-    (property "MANUFACTURE PART NO" "M7")
     (property "MANUFACTURER" "Diotec Semiconductor")
+    (property "MANUFACTURER PART NO" "M7")
     (property "PACKAGE" "DO-214AC, SMA")
     (property "SUPPLIER" "DIGIKEY")
@@
       (net 5 "Net-(D2-K)") (pinfunction "K") (pintype "passive"))
     (pad "2" smd roundrect (at 1.525 0.125 180) (size 1.25 1.75) (layers "F.Cu" "F.Paste" "F.Mask") (roundrect_rratio 0.2)
-      (net 6 "/10V_OUT_P") (pinfunction "A") (pintype "passive"))
+      (net 6 "/12V_OUT_P") (pinfunction "A") (pintype "passive"))
     (model "${KIPRJMOD}/3D models/D2 -220AA-SMP.step"
       (offset (xyz 0 0 0))
@@
     (at 86.63 57.59)
     (tags "ERJ-P08J150V ")
-    (property "MANUFACTURE" "PANASONIC")
-    (property "MANUFACTURE PART NO" "ERJ-P08J150V")
+    (property "MANUFACTURER" "PANASONIC")
+    (property "MANUFACTURER PART NO" "ERJ-P08J150V")
     (property "PACKAGE" "1206")
     (property "SUPPLIER" "DIGIKEY")
@@
     (at 90.3216 66.93 180)
     (tags "DR127-102-R ")
-    (property "MANUFACTURE " "Eaton - Electronics Division")
+    (property "MANUFACTURER" "Eaton - Electronics Division")
     (property "MANUFACTURER PART NO" "DR127-102-R")
     (property "PACKAGE" ".")
@@
       (net 3 "Net-(D1-K)") (pinfunction "1") (pintype "passive"))
     (pad "2" smd rect (at 4.9784 0 180) (size 3.8608 5.5118) (layers "F.Cu" "F.Paste" "F.Mask")
-      (net 6 "/10V_OUT_P") (pinfunction "2") (pintype "passive"))
+      (net 6 "/12V_OUT_P") (pinfunction "2") (pintype "passive"))
     (zone (net 0) (net_name "") (layer "F.Cu") (hatch full 0.508)
       (connect_pads (clearance 0))
@@
     (descr "CP, Radial series, Radial, pin pitch=5.00mm, , diameter=10mm, Electrolytic Capacitor")
     (tags "CP Radial series Radial pin pitch 5.00mm  diameter 10mm Electrolytic Capacitor")
-    (property "MANUFACTURE" "Cornell Dubilier Knowles")
+    (property "MANUFACTURER" "Cornell Dubilier Knowles")
     (property "MANUFACTURER PART NO" "106CKS450MLU")
-    (property "PACKAGE " "RADIAL/THT")
+    (property "PACKAGE" "RADIAL/THT")
     (property "SUPPLIER" "DIGIKEY")
     (property "SUPPLIER PART NO" "1572-1650-ND")
@@
     (descr "Capacitor SMD 1206 (3216 Metric), square (rectangular) end terminal, IPC_7351 nominal, (Body size source: IPC-SM-782 page 76, https://www.pcb-3d.com/wordpress/wp-content/uploads/ipc-sm-782a_amendment_1_and_2.pdf), generated with kicad-footprint-generator")
     (tags "capacitor")
-    (property "MANUFACTURE PART NO" "UMF325B7104KNHT")
     (property "MANUFACTURER" "TAIYO YUDEN")
+    (property "MANUFACTURER PART NO" "UMF325B7104KNHT")
     (property "PACKAGE" "1206")
     (property "SUPPLIER" "MOUSER")
@@
   (gr_line (start 71 34.02) (end 115.73 34.02)
     (stroke (width 0.05) (type default)) (layer "Edge.Cuts"))
+  (gr_text "GND" (at 71.31 53.06 -90) (layer "F.SilkS")
+    (effects (font (size 1 1) (thickness 0.1)) (justify left bottom))
+  )
+  (gr_text "HV_IN" (at 71.41 58.3 -90) (layer "F.SilkS")
+    (effects (font (size 1 1) (thickness 0.1)) (justify left bottom))
+  )
+  (gr_text "12V" (at 71.42 47.55 -90) (layer "F.SilkS")
+    (effects (font (size 1 1) (thickness 0.1)) (justify left bottom))
+  )
   (segment (start 106.06 50.320908) (end 105.140908 51.24) (width 0.25) (layer "F.Cu") (net 1))
   (segment (start 85.48 52.72) (end 88 55.24) (width 0.25) (layer "F.Cu") (net 1))
