File: UC28881  WORK.kicad_sch (KiCad schematic)
At the start: 18 parts, among them J1 Screw_Terminal_01x02, J2 Screw_Terminal_01x02, U1 UCC28881

Commit message: Updated PCB
Parts:
- removed CL1: 330u, CL1:CAP_UAQ_18X20_NCH, symbol Device:C_Polarized_Small
- removed D3: 1N5819, Diode_THT:D_DO-41_SOD81_P10.16mm_Horizontal, symbol Diode:1N5819
- removed J1, J2: Screw_Terminal_01x02, TerminalBlock_Phoenix:TerminalBlock_Phoenix_MKDS-1,5-2_1x02_P5.00mm_Horizontal, symbol Connector:Screw_Terminal_01x02
- removed TVS1: D_Zener, TVS1:1.5KESeries_LTF, symbol Device:D_Zener
- added H1, H2, H3, H4: MountingHole, MountingHole:MountingHole_3.2mm_M3_DIN965, symbol Mechanical:MountingHole
- added J1: Screw_Terminal_01x03, TerminalBlock_Phoenix:TerminalBlock_Phoenix_MKDS-1,5-3-5.08_1x03_P5.08mm_Horizontal, symbol Connector:Screw_Terminal_01x03
- C1: footprint Capacitor_THT:CP_Radial_D12.5mm_P7.50mm -> Capacitor_THT:CP_Radial_D10.0mm_P5.00mm
- D1: footprint Diode_THT:D_DO-35_SOD27_P7.62mm_Horizontal -> D1:SMA_STM-M
- D2: value SS1P3L -> M7; footprint Diode_SMD:D_1206_3216Metric -> D2:D2
- RFB1: footprint 10k resistor:10k RES_3540_TEC-M -> 10k resistor:10k RESC1005X35N
- RFB2: value 87.7K -> 110k; footprint 88.7k resistor:ERJS1T_U1T__2512_ -> 110k resistor:110k RESC1005X35N
- Rf1: footprint Resistor_THT:R_Axial_DIN0922_L20.0mm_D9.0mm_P30.48mm_Horizontal -> RF:ERJUP6; POWER 10W -> 0.5W
Connections:
- net 10V_OUT_P: now also J1.1 (Pin_1)
- net GND: now also J1.2 (Pin_2)
- net HV_IN_P: now also J1.3 (Pin_3)

Commit message: Updated project files and fixed latest edits
Parts:
- L1: footprint L1 1MH:IND_EPCOS_B82472G6_EPC -> L1 1MH:L_Wurth_WE-PD2HV-7850; ORDER CODE (none) -> 76877530; PART NUMBER 495-5675-6-ND -> (none)
- RFB1: footprint 10k resistor:10k RESC1005X35N -> 10k resistor:RESC3116X65N; PART NUMBER (none) -> CR2010-FX-1002ELF
- RFB2: footprint 110k resistor:110k RESC1005X35N -> 110k resistor:RESC3216X75N; part number (none) -> CR1206-JW-114ELF
- Rf1: value 10 -> 15; footprint RF:ERJUP6 -> RF:RF1 RC1206N_PAN-M
Changed lines of the file:
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@@
       (effects (font (size 1.27 1.27)))
     )
-    (property "Value" "10" (at 38.1 52.07 90)
-      (effects (font (size 1.27 1.27)))
-    )
-    (property "Footprint" "RF:ERJUP6" (at 38.1 57.658 90)
-      (effects (font (size 1.27 1.27)) hide)
-    )
-    (property "Datasheet" "https://www.mouser.com/ProductDetail/Panasonic/ERJ-UP6F14R0V?qs=sGAEpiMZZMtlubZbdhIBICtThL%252B6LvXHTYktNu5WFLk%3D" (at 38.1 55.88 0)
+    (property "Value" "15" (at 38.1 52.07 90)
+      (effects (font (size 1.27 1.27)))
+    )
+    (property "Footprint" "RF:RF1  RC1206N_PAN-M" (at 38.1 57.658 90)
+      (effects (font (size 1.27 1.27)) hide)
+    )
+    (property "Datasheet" "https://www.digikey.com/en/products/detail/panasonic-electronic-components/ERJ-P08J150V/525576?curr=usd&utm_campaign=buynow&utm_medium=aggregator&utm_source=octopart" (at 38.1 55.88 0)
       (effects (font (size 1.27 1.27)) hide)
     )
@@
       (effects (font (size 1.27 1.27)) (justify right))
     )
-    (property "Footprint" "10k resistor:10k RESC1005X35N" (at 187.198 74.93 90)
-      (effects (font (size 1.27 1.27)) hide)
-    )
-    (property "Datasheet" "https://www.digikey.com/en/products/detail/te-connectivity-passive-product/CRGCQ0402F10K/8577471?curr=usd&utm_campaign=buynow&utm_medium=aggregator&utm_source=octopart" (at 185.42 74.93 0)
+    (property "Footprint" "10k resistor:RESC3116X65N" (at 187.198 74.93 90)
+      (effects (font (size 1.27 1.27)) hide)
+    )
+    (property "Datasheet" "https://www.digikey.com/en/products/detail/bourns-inc/CR2010-FX-1002ELF/21774723?curr=usd&utm_campaign=buynow&utm_medium=aggregator&utm_source=octopart" (at 185.42 74.93 0)
       (effects (font (size 1.27 1.27)) hide)
     )
@@
     )
     (property "Sim.Pins" "1=+ 2=-" (at 185.42 74.93 0)
+      (effects (font (size 1.27 1.27)) hide)
+    )
+    (property "PART NUMBER" "CR2010-FX-1002ELF" (at 185.42 74.93 0)
       (effects (font (size 1.27 1.27)) hide)
     )
@@
       (effects (font (size 1.27 1.27)) (justify left))
     )
-    (property "Footprint" "110k resistor:110k RESC1005X35N" (at 207.01 58.928 90)
-      (effects (font (size 1.27 1.27)) hide)
-    )
-    (property "Datasheet" "https://www.digikey.com/en/products/detail/te-connectivity-passive-product/CPF0402B110KE1/2729564?curr=usd&utm_campaign=buynow&utm_medium=aggregator&utm_source=octopart" (at 207.01 57.15 0)
+    (property "Footprint" "110k resistor:RESC3216X75N" (at 207.01 58.928 90)
+      (effects (font (size 1.27 1.27)) hide)
+    )
+    (property "Datasheet" "https://www.digikey.com/en/products/detail/bourns-inc/CR1206-JW-114ELF/3785526" (at 207.01 57.15 0)
       (effects (font (size 1.27 1.27)) hide)
     )
@@
       (effects (font (size 1.27 1.27)) hide)
     )
+    (property "part number" "CR1206-JW-114ELF" (at 207.01 57.15 0)
+      (effects (font (size 1.27 1.27)) hide)
+    )
     (pin "1")
     (pin "2")
@@
       (effects (font (size 1.27 1.27)))
     )
-    (property "Footprint" "L1 1MH:IND_EPCOS_B82472G6_EPC" (at 93.98 55.88 0)
-      (effects (font (size 1.27 1.27)) hide)
-    )
-    (property "Datasheet" "https://www.digikey.com/en/products/detail/tdk-electronics-inc/B82472G6105M000/4245753?curr=usd" (at 93.98 55.88 0)
-      (effects (font (size 1.27 1.27)) hide)
-    )
-    (property "PART NUMBER" "495-5675-6-ND" (at 93.98 55.88 0)
-      (effects (font (size 1.27 1.27)) hide)
-    )
+    (property "Footprint" "L1 1MH:L_Wurth_WE-PD2HV-7850" (at 93.98 55.88 0)
+      (effects (font (size 1.27 1.27)) hide)
+    )
+    (property "Datasheet" "https://www.we-online.com/en/components/products/WE-PD2-HV#/articles/WE-PD2-HV-7850" (at 93.98 55.88 0)
+      (effects (font (size 1.27 1.27)) hide)
+    )
+    (property "ORDER CODE" "76877530" (at 93.98 55.88 0)
+      (effects (font (size 1.27 1.27)) hide)
+    )

Commit message: update
Parts:
- added COUT1: 47UF, Capacitor_SMD:C_1206_3216Metric_Pad1.33x1.80mm_HandSolder, symbol Device:C
- D1: value 1N4148 -> STTH1R06A
- renumbered H4 to H1, H1 to H4
Connections:
- net 10V_OUT_P: now also COUT1.1
- net GND: now also COUT1.2
Changed lines of the file:
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@@
   (junction (at 154.94 62.23) (diameter 0) (color 0 0 0 0)
+  )
+  (junction (at 245.11 88.9) (diameter 0) (color 0 0 0 0)
   )
   (junction (at 135.89 88.9) (diameter 0) (color 0 0 0 0)
@@
     (stroke (width 0) (type default))
   )
-  (wire (pts (xy 241.3 88.9) (xy 254 88.9))
+  (wire (pts (xy 241.3 88.9) (xy 245.11 88.9))
     (stroke (width 0) (type default))
   )
@@
     (stroke (width 0) (type default))
   )
+  (wire (pts (xy 135.89 88.9) (xy 170.18 88.9))
+    (stroke (width 0) (type default))
+  )
   (wire (pts (xy 24.13 116.84) (xy 48.26 116.84))
     (stroke (width 0) (type default))
@@
     (stroke (width 0) (type default))
   )
+  (wire (pts (xy 245.11 88.9) (xy 254 88.9))
+    (stroke (width 0) (type default))
+  )
   (wire (pts (xy 274.32 91.44) (xy 274.32 99.06))
     (stroke (width 0) (type default))
@@
     (stroke (width 0) (type default))
   )
+  (wire (pts (xy 245.11 88.9) (xy 245.11 97.79))
+    (stroke (width 0) (type default))
+  )
   (wire (pts (xy 170.18 77.47) (xy 170.18 88.9))
     (stroke (width 0) (type default))
@@
   )
   (wire (pts (xy 41.91 55.88) (xy 77.47 55.88))
-    (stroke (width 0) (type default))
-  )
-  (wire (pts (xy 170.18 88.9) (xy 135.89 88.9))
     (stroke (width 0) (type default))
   )
@@
   (label "10V_OUT_P" (at 274.32 91.44 90) (fields_autoplaced)
     (effects (font (size 1.27 1.27)) (justify left bottom))
+  )
+  (label "GND" (at 245.11 105.41 270) (fields_autoplaced)
+    (effects (font (size 1.27 1.27)) (justify right bottom))
   )
   (label "HV_IN_P" (at 24.13 55.88 180) (fields_autoplaced)
@@
       (effects (font (size 1.27 1.27)) (justify left))
     )
-    (property "Value" "1N4148" (at 138.43 100.33 90)
+    (property "Value" "STTH1R06A" (at 138.43 100.33 90)
       (effects (font (size 1.27 1.27)) (justify left))
     )
@@
     )
   )
+  (symbol (lib_id "Device:C") (at 245.11 101.6 0) (unit 1)
+    (in_bom yes) (on_board yes) (dnp no) (fields_autoplaced)
+    (property "Reference" "COUT1" (at 248.92 100.33 0)
+      (effects (font (size 1.27 1.27)) (justify left))
+    )
+    (property "Value" "47UF" (at 248.92 102.87 0)
+      (effects (font (size 1.27 1.27)) (justify left))
+    )
+    (property "Footprint" "Capacitor_SMD:C_1206_3216Metric_Pad1.33x1.80mm_HandSolder" (at 246.0752 105.41 0)
+      (effects (font (size 1.27 1.27)) hide)
+    )
+    (property "Datasheet" "https://product.tdk.com/system/files/dam/doc/product/capacitor/ceramic/mlcc/catalog/mlcc_commercial_general_en.pdf" (at 245.11 101.6 0)
+      (effects (font (size 1.27 1.27)) hide)
+    )
+    (property "PART NUMBER" "C3216X5R1C476M160AB" (at 245.11 101.6 0)
+      (effects (font (size 1.27 1.27)) hide)
+    )
+    (pin "1")
+    (pin "2")
+    (instances
+      (project "UC28881  WORK"
+        (path "/02261b3b-0ab5-411c-b90d-2981c1ef32c1"
+          (reference "COUT1") (unit 1)
+        )
+      )
+    )
+  )
   (symbol (lib_id "Mechanical:MountingHole") (at 33.02 78.74 0) (unit 1)
     (in_bom yes) (on_board yes) (dnp no) (fields_autoplaced)
@@
   (symbol (lib_id "Mechanical:MountingHole") (at 265.43 59.69 0) (unit 1)
     (in_bom yes) (on_board yes) (dnp no) (fields_autoplaced)
-    (property "Reference" "H1" (at 267.97 58.42 0)
+    (property "Reference" "H4" (at 267.97 58.42 0)
       (effects (font (size 1.27 1.27)) (justify left))
     )
@@
       (project "UC28881  WORK"
         (path "/02261b3b-0ab5-411c-b90d-2981c1ef32c1"
-          (reference "H1") (unit 1)
+          (reference "H4") (unit 1)
         )
       )
@@
   (symbol (lib_id "Mechanical:MountingHole") (at 30.48 86.36 0) (unit 1)
     (in_bom yes) (on_board yes) (dnp no) (fields_autoplaced)
-    (property "Reference" "H4" (at 33.02 85.09 0)
+    (property "Reference" "H1" (at 33.02 85.09 0)
       (effects (font (size 1.27 1.27)) (justify left))
     )
@@
       (project "UC28881  WORK"
         (path "/02261b3b-0ab5-411c-b90d-2981c1ef32c1"
-          (reference "H4") (unit 1)
-        )
-      )
+          (reference "H1") (unit 1)
+        )
+      )

Commit message: ADDED BOM
Parts:
- C1: MANUFACTURER (none) -> Cornell Dubilier Knowles; MANUFACTURER PART NO (none) -> 106CKS450MLU; PACKAGE (none) -> RADIAL/THT; PART NUMBER 1572-1650-ND -> (none); SUPPLIER (none) -> DIGIKEY; SUPPLIER PART NO (none) -> 1572-1650-ND; VOLTAGE 450V -> (none)
- C2: footprint C2:CAPC3225X88N -> Capacitor_SMD:C_1206_3216Metric; MANUFACTURER (none) -> KYOCERA AVX; MANUFACTURER PART NO (none) -> 12065C104JAT2A; MANUFACTURER PART NUMBER 495-3216-ND -> (none); PACKAGE (none) -> 1206; SUPPLIER (none) -> MOUSER; SUPPLIER PART NO (none) -> 581-12065C104J
- C3: footprint C3:CAP_ECHU1H104GX9 -> Capacitor_SMD:C_1206_3216Metric; MANUFACTURER (none) -> TAIYO YUDEN; MANUFACTURER PART NO (none) -> UMF325B7104KNHT; MANUFACTURER PART NUMBER 587-2835-6-ND -> (none); PACKAGE (none) -> 1206; SUPPLIER (none) -> MOUSER; SUPPLIER PART NO (none) -> PCF1552CT-ND; VOLTAGE 10v -> (none)
- C4: footprint C4:CAP_ECHU1H104GX9 -> Capacitor_SMD:C_1206_3216Metric; MANUFACTURER (none) -> KEMET; MANUFACTURER PART NO (none) -> C1206C153K5RACTU; MANUFACTURER PART NUMBER 587-2835-6-ND -> (none); PACKAGE (none) -> 1206; SUPPLIER (none) -> DIGIKEY; SUPPLIER PART NO (none) -> 399-C1206C153K5RACTUCT-ND; VOLTAGE 10v -> (none)
- CBULK1: MANUFACTURER (none) -> Cornell Dubilier Knowles; MANUFACTURER PART NO (none) -> 106CKS450MLU; PACKAGE (none) -> Radial /THT; PART NUMBER 1572-1650-ND -> (none); SUPPLIER (none) -> DIGIKEY; SUPPLIER PART NO (none) -> 1572-1650-ND; VOLTAGE 450V -> (none)
- COUT1: MANUFACTURER (none) -> TDK Corporation; MANUFACTURER PART NO (none) -> C3216X5R1C476M160AB; PACKAGE (none) -> 1206; PART NUMBER C3216X5R1C476M160AB -> (none); SUPPLIER (none) -> DIGIKEY; SUPPLIER PART NO (none) -> 445-6003-1-ND
- D1: MANUFACTURER (none) -> STMicroelectronics; MANUFACTURER PART NO (none) -> STTH1R06A; PACKAGE (none) -> DO-214AC, SMA; SUPPLIER (none) -> DIGIKEY; SUPPLIER PART NO (none) -> 497-3765-1-ND
- D2: MANUFACTURER (none) -> Diotec Semiconductor; MANUFACTURER PART NO (none) -> M7; PACKAGE (none) -> DO-214AC, SMA; SUPPLIER (none) -> DIGIKEY; SUPPLIER PART NO (none) -> 4878-M7DKR-ND
- H1, H2, H3, H4: now left out of the parts list
- J1: MANUFACTURER (none) -> PHOENIX CONTACT; MANUFACTURER PART NO (none) -> .; PACKAGE (none) -> .; SUPPLIER (none) -> .; SUPPLIER PART NO (none) -> .
- L1: MANUFACTURER (none) -> .; MANUFACTURER PART NO (none) -> 76877530; ORDER CODE 76877530 -> (none); SUPPLIER (none) -> .; SUPPLIER PART NO (none) -> .
- L2: MANUFACTURER (none) -> Eaton - Electronics Division; MANUFACTURER PART NO (none) -> DR127-102-R; PACKAGE (none) -> .; SUPPLIER (none) -> DIGIKEY; SUPPLIER PART NO (none) -> 513-1217-1-ND
- RFB1: MANUFACTURER (none) -> Bourns Inc.; MANUFACTURER PART NO (none) -> CR2010-FX-1002ELF; PACKAGE (none) -> 2010; PART NUMBER CR2010-FX-1002ELF -> (none); SUPPLIER (none) -> DIGIKEY; SUPPLIER PART NO (none) -> 118-CR2010-FX-1002ELFCT-ND
- RFB2: MANUFACTURER (none) -> Bourns Inc.; MANUFACTURER PART NO (none) -> CR1206-JW-114ELF; PACKAGE (none) -> 1206; SUPPLIER (none) -> DIGIKEY; SUPPLIER PART NO (none) -> 118-CR1206-JW-114ELFCT-ND; part number CR1206-JW-114ELF -> (none)
- Rf1: MANUFACTURER (none) -> PANASONIC; MANUFACTURER PART NO (none) -> ERJ-P08J150V; PACKAGE (none) -> 1206; POWER 0.5W -> (none); SUPPLIER (none) -> DIGIKEY; SUPPLIER PART NO (none) -> P15ALCT-ND
- U1: MANUFACTURER (none) -> TEXAS INSTRUMENTS; MANUFACTURER PART NO (none) -> UCC28810D; PACKAGE (none) -> 8-SOIC; SUPPLIER (none) -> DIGIKEY; SUPPLIER PART NO (none) -> 296-27162-5-ND

Commit message: update
Connections:
- net 10V_OUT_P renamed 12V_OUT_P
Changed lines of the file:
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@@
     (stroke (width 0) (type default))
   )
-  (label "10V_OUT_P" (at 274.32 91.44 90) (fields_autoplaced)
+  (label "12V_OUT_P" (at 274.32 91.44 90) (fields_autoplaced)
     (effects (font (size 1.27 1.27)) (justify left bottom))
   )
@@
     (effects (font (size 1.27 1.27)) (justify right bottom))
   )
-  (label "10V_OUT_P" (at 254 88.9 0) (fields_autoplaced)
+  (label "12V_OUT_P" (at 254 88.9 0) (fields_autoplaced)
     (effects (font (size 1.27 1.27)) (justify left bottom))
   )
